File: hardware/RUDRAKINUXIS_Lite.kicad_sch (KiCad schematic)
At the start: 0 parts

Commit message: I uploaded all latest files to GitHub
Other:
- title: RUDRAKINUXIS_Lite - 500W/600W 4S-6S FOC BLDC Speed Controller -> RUDRAKINUXIS_Lite - 4S-6S (12V-25.6V) High-Performance FOC BLDC Speed Controller
Changed lines of the file:
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@@
 (kicad_sch
-  (version 20260101)
-  (generator "RUDRAKINUXIS_Setup")
+  (version 20240108)
+  (generator "eeschema")
   (generator_version "10.0")
   (paper "A3")
   (title_block
-    (title "RUDRAKINUXIS_Lite - 500W/600W 4S-6S FOC BLDC Speed Controller")
-    (date "2026-09-10")
-    (rev "v1.0")
+    (title "RUDRAKINUXIS_Lite - 4S-6S (12V-25.6V) High-Performance FOC BLDC Speed Controller")
+    (date "2026-09-29")
+    (rev "v1.1")
     (company "Engineered by Ravi Kachhwaha")
-    (comment 1 "Operating Voltage: 12V-24V Nominal (4S-6S LiPo, 28V Max)")
-    (comment 2 "Dual Control: DroneCAN/DShot FC Link + Isolated USB-C Diagnostics + Hardware Test Mode")
+    (comment 1 "Rating: 60A Cont (1.5kW) / 80A Burst (2.0kW) / 100A Boost (2.5kW) / 120A Transient (3.0kW)")
+    (comment 2 "Gate Driver: Texas Instruments DRV8300DPWR (100V 1.5A Peak, Integrated Bootstrap Diodes)")
+    (comment 3 "Power Tree: LMR36510 (10V Gate Rail) -> L78L05 (5V CAN VCC) -> AP2112K (3.3V Logic LDO)")
+    (comment 4 "DC-Link Bulk: Panasonic EEU-FR1H102 1000uF 50V Low-ESR Radial Can (D16mm P7.5mm On-Board)")
+  )
+  (sheet_instances
+    (path "/"
+      (page "1")
+    )
   )
 )

Commit message: Uploading latest files, 50% work done in schematic
Parts:
- added C11, C12, C34, C_MCU2, C_MCU3, C_MCU4: 100nF, Capacitor_SMD:C_0603_1608Metric, symbol Device:C
- added C2: EEUFR1H102, easyeda2kicad:CAP_16 X 25_PAN, symbol easyeda2kicad:EEUFR1H102
- added C20, C21, C22: 10uF, Capacitor_SMD:C_1206_3216Metric, symbol Device:C
- added C24, C25, C26, C28, C33, C37: 1uF, Capacitor_SMD:C_0603_1608Metric, symbol Device:C
- added D1: SMCJ28A, easyeda2kicad:DIODE_DO-214AC, symbol easyeda2kicad:SMCJ28A
- added D2: SS14, Diode_SMD:D_SMA, symbol Diode:SS14
- added FB1: 600R, Inductor_SMD:L_0603_1608Metric, symbol easyeda2kicad:BLM18KG601SN1D
- added J1: USB4105-GF-A, easyeda2kicad:TYPE-C-SMD_SBC-160S1A-20-S412, symbol easyeda2kicad:USB4105-GF-A
- added J2: SM06B-SRSS-TB, easyeda2kicad:CONN-SMD_SM06B-SRSS-TB-LF-SN, symbol easyeda2kicad:SM06B-SRSS-TB
- added L1: 47uH, easyeda2kicad:IND-SMD_L10.2-W10.0, symbol easyeda2kicad:CDRH105RNP-470NC
- added LED1: Green, LED_SMD:LED_0603_1608Metric, symbol Device:LED
- added LED2: Blue, LED_SMD:LED_0603_1608Metric, symbol Device:LED
- added Q1, Q2, Q3, Q4, Q5, Q6: NTMFS5H600NLT1G, easyeda2kicad:DFN-5_L5.9-W4.9-P1.27-LS6.2-BL_CASE-488AA, symbol easyeda2kicad:NTMFS5H600NLT1G
- added R4, R5: 5.1k, Resistor_SMD:R_0603_1608Metric, symbol Device:R
- added R6: 100k, Resistor_SMD:R_0603_1608Metric, symbol Device:R
- added R7: 11k, Resistor_SMD:R_0603_1608Metric, symbol Device:R
- added R8, R9: 1k, Resistor_SMD:R_0603_1608Metric, symbol Device:R
- added R_PD6_BOOT: R10k, Resistor_SMD:R_0603_1608Metric, symbol Device:R
- added SW1: B3S-1000P, easyeda2kicad:KEY-SMD_4P-L6.6-W6.0-P4.50-LS9.0-BR, symbol easyeda2kicad:B3S-1000P
- added TH1: THERMISTOR NTC 10KOHM 3380K 0603, Resistor_SMD:R_0603_1608Metric, symbol Device:Thermistor_NTC
- added U1: STM32G431CBU6, easyeda2kicad:VQFN-48_L7.0-W7.0-P0.50-BL-EP5.5, symbol easyeda2kicad:STM32G431CBU6
- added U2: DRV8300DPWR, easyeda2kicad:TSSOP-20_L6.5-W4.4-P0.65-LS6.4-BL, symbol easyeda2kicad:DRV8300DPWR
- added U3: LMR36510ADDAR, easyeda2kicad:SOP-8_L5.0-W4.0-P1.27-LS6.2-BL-EP, symbol easyeda2kicad:LMR36510ADDAR
- added U4: L78L05ABUTR, easyeda2kicad:SOT-89-3_L4.5-W2.5-P1.50-LS4.2-TL, symbol easyeda2kicad:L78L05ABUTR
- added U5: AP2112K-3.3, easyeda2kicad:SOT-25-5_L2.9-W1.6-P0.95-LS2.8-BL, symbol easyeda2kicad:AP2112K-3.3TRG1
- added U6: CP2102N, easyeda2kicad:QFN-24_L4.0-W4.0-P0.50-TL-EP2.6, symbol easyeda2kicad:CP2102N-A02-GQFN24R
- added U7: TJA1051T/3,118, easyeda2kicad:SOIC-8_L4.9-W3.9-P1.27-LS6.0-BL, symbol easyeda2kicad:TJA1051T_3,118
- added U8: USBLC6-2SC6, easyeda2kicad:SOT-23-6_L2.9-W1.6-P0.95-LS2.8-BL, symbol easyeda2kicad:USBLC6-2SC6
- added U9: ESDCAN24-2BLY, easyeda2kicad:SOT_24-2BLY_STM, symbol easyeda2kicad:ESDCAN24-2BLY
Connections:
- new net: C_MCU2.1, U1.23 (VDD)
- new net: C_MCU3.1, U1.35 (VDD)
- new net: C_MCU4.1, U1.48 (VDD)
- new net: LED1.2 (A), R8.2
- new net: LED2.2 (A), R9.2
- new net +10V_GATE: C21.2, C22.2, C25.1, L1.2, R6.1, U4.3 (VIN)
- new net +3V3_SYS: C11.2, C37.1, FB1.1, R8.1, U1.1 (VBAT), U5.5 (VOUT), U6.5 (VIO), U6.6 (VDD), U6.9 (RSTb)
- new net +5V_AUX: C24.1, C26.1, D2.1 (K), U4.1 (VOUT), U5.1 (VIN), U5.3 (EN), U6.7 (VREGIN), U6.8 (VBUS)
- new net BEMF_U: U1.13 (PA5)
- new net BEMF_V: U1.14 (PA6)
- new net BEMF_W: U1.15 (PA7)
- new net BIDIR_DSHOT: J2.4, U1.12 (PA4)
- new net BOOT0_GND: R_PD6_BOOT.1, U1.46 (PB8-BOOT0)
- new net BOOT_10V: C34.2, U3.7 (BOOT)
- new net CAN_H: J2.5
- new net CAN_L: J2.6
- new net CAN_RX: U1.24 (PB11)
- new net CAN_TX: U1.25 (PB12)
- new net DSHOT_IN: J2.2, U1.33 (PA11)
- new net GND: C11.1, C12.2, C20.2, C21.1, C22.1, C24.2, C25.2, C26.2, C28.1, C33.1, C37.2, C_MCU2.2, C_MCU3.2, C_MCU4.2, J1.1 (EH), J1.2 (EH), J1.3 (EH), J1.4 (EH), J1.A1 (GND), J1.A12 (GND), J1.B1 (GND), J1.B12 (GND), J2.1, J2.7, J2.8, LED1.1 (K), LED2.1 (K), R4.2, R5.1, R7.1, R_PD6_BOOT.2, U1.49 (VSS), U3.1 (PGND), U3.9 (PAD), U4.2 (GND), U5.2 (GND), U6.18 (CTS), U6.2 (GND), U6.25 (GND), U8.2
- new net IN_HU: U1.30 (PA8)
- new net IN_HV: U1.31 (PA9)
- new net IN_HW: U1.32 (PA10)
- new net IN_LU: U1.19 (PB2)
- new net IN_LV: U1.17 (PB0)
- new net IN_LW: U1.18 (PB1)
- new net ISENSE_U: U1.8 (PA0)
- new net ISENSE_V: U1.9 (PA1)
- new net ISENSE_W: U1.16 (PC4)
- new net MCU_RESET: C12.1, U1.7 (PG10-NRST)
- new net MCU_UART_RX: U1.11 (PA3), U6.21 (TXD)
- new net MCU_UART_TX: J2.3, U1.10 (PA2), U6.20 (RXD)
- new net STATUS_LED: R9.1, U1.2 (PC13)
- new net SW1_TEST: U1.38 (PA15)
- new net SWCLK: U1.37 (PA14)
- new net SWDIO: U1.36 (PA13)
- new net SW_10V: C34.1, L1.1, U3.8 (SW)
- new net TEMP_SENSE: U1.22 (PB10)
- new net USB_CC1: J1.A5 (CC1), R4.1
- new net USB_CC2: J1.B5 (CC2), R5.2
- new net USB_DN: J1.A7 (DN1), J1.B7 (DN2), U6.4 (D-), U8.3, U8.4
- new net USB_DP: J1.A6 (DP1), J1.B6 (DP2), U6.3 (D+), U8.1, U8.6
- new net VBAT_SENSE: U1.27 (PB14)
- new net VBUS_RAW: D2.2 (A), J1.A4 (VBUS), J1.A9 (VBUS), J1.B4 (VBUS), J1.B9 (VBUS), U8.5
- new net VCC_10V: C33.2, U3.6 (VCC)
- new net VDDA: C28.2, FB1.2, U1.20 (VREF+), U1.21 (VDDA)
- new net V_BAT: C20.1, U3.2 (VIN), U3.3 (EN)
- new net V_FB_10V: R6.2, R7.2, U3.5 (FB)
- no-connect marks 0 -> 33

Commit message: Uploading latest files after 100% schematic done
Parts:
- removed SW1: B3S-1000P, easyeda2kicad:KEY-SMD_4P-L6.6-W6.0-P4.50-LS9.0-BR, symbol easyeda2kicad:B3S-1000P
- added C10, C16, C17, C8, C9: 100nF, Capacitor_SMD:C_0603_1608Metric, symbol Device:C
- added C19, C2, C3, C4, C5, C6, C7: 10uF, Capacitor_SMD:C_1206_3216Metric, symbol Device:C
- added C29, C30, C31, C32, C33, C34: 1nF, Capacitor_SMD:C_0603_1608Metric, symbol Device:C
- added D3: SS14, Diode_SMD:D_SMA, symbol Device:D_Schottky
- added PAD1: BAT+, Custom_Pads:Pad_10x7mm_WireHole, symbol Connector:TestPoint_Square
- added PAD2: BAT-, Custom_Pads:Pad_10x7mm_WireHole, symbol Connector:TestPoint_Square
- added PAD3: PHASE_U, Custom_Pads:Pad_10x7mm_WireHole, symbol Connector:TestPoint_Square
- added PAD4: PHASE_V, Custom_Pads:Pad_10x7mm_WireHole, symbol Connector:TestPoint_Square
- added PAD5: PHASE_W, Custom_Pads:Pad_10x7mm_WireHole, symbol Connector:TestPoint_Square
- added R1, R2, R3: 0.5m, Resistor_SMD:R_2512_6332Metric, symbol Device:R
- added R10, R11, R12, R13, R14, R15, R16, R18: 10k, Resistor_SMD:R_0603_1608Metric, symbol Device:R
- added R12, R14, R16, R19, R20, R21, R22: 33k, Resistor_SMD:R_0603_1608Metric, symbol Device:R
- added R23, R24, R25, R26: 3.3k, Resistor_SMD:R_0603_1608Metric, symbol Device:R
- added R27, R28, R29, R30, R31, R32: 100R, Resistor_SMD:R_0603_1608Metric, symbol Device:R
- added R39: 120R, Resistor_SMD:R_0805_2012Metric, symbol Device:R
- added R4, R5, R6, R7, R8, R9: 10, Resistor_SMD:R_0603_1608Metric, symbol Device:R
- added R40: 33k, Resistor_SMD:R_1206_3216Metric, symbol Device:R
- added SW1: B3S-1000P, symbol Switch:SW_Push
- C1: renamed from C2; value EEUFR1H102 -> 1000uF
- R17: renamed from R_PD6_BOOT; value R10k -> 10k
- TH1: value THERMISTOR NTC 10KOHM 3380K 0603 -> 10k NTC
- renumbered C_MCU2 to C13, C_MCU3 to C14, C_MCU4 to C15, C34 to C18, C33 to C23, C25 to C24, C24 to C25, C37 to C27, R4 to R33, R5 to R34, R6 to R35, R7 to R36, R8 to R37, R9 to R38
Connections:
- net +10V_GATE: now also U2.7 (GVDD), C19.2
- net +3V3_SYS: now also C13.1, C14.1, C15.1, U1.23 (VDD), U1.35 (VDD), U1.48 (VDD), U7.5 (VIO), C17.2, R18.2, SW1.1
- net +5V_AUX: now also U7.3 (VCC), C16.2, D3.2 (A); no longer C26.1, D2.1 (K), U5.1 (VIN), U5.3 (EN), U6.7 (VREGIN), U6.8 (VBUS)
- net BEMF_U: now also C29.1, R12.1, R19.2, R23.1
- net BEMF_V: now also C30.1, R14.1, R20.2, R24.1
- net BEMF_W: now also C31.1, R16.1, R21.2, R25.1
- net CAN_H: now also U7.7 (CANH), U9.1, R39.1
- net CAN_L: now also U7.6 (CANL), U9.2, R39.2
- net CAN_RX: now also U7.4 (RXD)
- net CAN_TX: now also U7.1 (TXD)
- net GND: now also C1.2, D1.2, TH1.2, U2.8 (GND), U7.2 (GND), U7.8 (S), U9.3, C16.1, C17.1, C19.1, C2.1, C29.2, C3.1, C30.2, C31.2, C32.2, C33.2, C34.2, C4.1, C5.1, C6.1, C7.1, PAD2.1, R1.2, R16.2, R2.2, R23.2, R24.2, R25.2, R26.2, R28.1, R28.2, R3.2, R30.1, R30.2, R32.1, R32.2, R40.2
- net IN_HU: now also U2.1 (INHA)
- net IN_HV: now also U2.2 (INHB)
- net IN_HW: now also U2.3 (INHC)
- net IN_LU: now also U2.4 (INLA)
- net IN_LV: now also U2.5 (INLB)
- net IN_LW: now also U2.6 (INLC)
- net ISENSE_U: now also C32.1, R27.2
- net ISENSE_V: now also C33.1, R29.2
- net ISENSE_W: now also C34.1, R31.2
- net SW1_TEST: now also R16.1, SW1.2
- net TEMP_SENSE: now also TH1.1, R18.1
- net VBAT_SENSE: now also R22.2, R26.1
- net VBUS_RAW: now also U6.8 (VBUS)
- net V_BAT: now also C1.1, D1.1, Q1.5 (D), Q3.5 (D), Q5.5 (D), C2.2, C3.2, C4.2, C5.2, C6.2, C7.2, PAD1.1, R22.1, R40.1
- net R1_Kelvin (+): now reaches Q2.1 (S)
- net R1_Kelvin (+): now also Q2.2 (S), Q2.3 (S), R1.1, R11.1, R27.1
- net at Q2.4 (G): now also R11.2, R5.2
- net MOTOR_U: now reaches Q2.5 (D)
- net MOTOR_U: now also Q1.1 (S), Q1.2 (S), Q1.3 (S), PAD3.1, R10.1, R19.1
- net MOTOR_V: now reaches Q3.1 (S)
- net MOTOR_V: now also Q3.2 (S), Q3.3 (S), Q4.5 (D), PAD4.1, R12.1, R20.1
- net at Q3.4 (G): now also R12.2, R6.2
- net at Q1.4 (G): now also R10.2, R4.2
- net R3_Kelvin (+): now reaches Q6.1 (S)
- net R3_Kelvin (+): now also Q6.2 (S), Q6.3 (S), R15.1, R3.1, R31.1
- net at Q6.4 (G): now also R15.2, R9.2
- net MOTOR_W: now reaches Q6.5 (D)
- net MOTOR_W: now also Q5.1 (S), Q5.2 (S), Q5.3 (S), PAD5.1, R14.1, R21.1
- net at Q5.4 (G): now also R14.2, R8.2
- net GATE_LV_DRV: now reaches U2.10 (GLB)
- net GATE_LV_DRV: now also R7.1
- net GATE_LU_DRV: now reaches U2.11 (GLA)
- net GATE_LU_DRV: now also R5.1
- net PHASE_W: now reaches U2.12 (SHC)
- net PHASE_W: now also C10.1, R16.2
- net GATE_HW_DRV: now reaches U2.13 (GHC)
- net GATE_HW_DRV: now also R8.1
- net BOOT_W: now reaches U2.14 (BSTC)
- net BOOT_W: now also C10.2
- net PHASE_V: now reaches U2.15 (SHB)
- net PHASE_V: now also C9.1, R14.2
- net GATE_HV_DRV: now reaches U2.16 (GHB)
- net GATE_HV_DRV: now also R6.1
- net BOOT_V: now reaches U2.17 (BSTB)
- net BOOT_V: now also C9.2
- net PHASE_U: now reaches U2.18 (SHA)
- net PHASE_U: now also C8.1, R12.2
- net GATE_HU_DRV: now reaches U2.19 (GHA)
- net GATE_HU_DRV: now also R4.1
- net BOOT_U: now reaches U2.20 (BSTA)
- net BOOT_U: now also C8.2
- net GATE_LW_DRV: now reaches U2.9 (GLC)
- net GATE_LW_DRV: now also R9.1
- net R2_Kelvin (+): now reaches Q4.1 (S)
- net R2_Kelvin (+): now also Q4.2 (S), Q4.3 (S), R13.1, R2.1, R29.1
- net at Q4.4 (G): now also R13.2, R7.2
- new net VBUS_ISO: C26.1, D2.1 (K), D3.1 (K), U5.1 (VIN), U5.3 (EN), U6.7 (VREGIN)
Other:
- company: Engineered by Ravi Kachhwaha -> Engineered and desinged by Ravi Kachhwaha
- title: RUDRAKINUXIS_Lite - 4S-6S (12V-25.6V) High-Performance FOC BLDC Speed Controller -> RUDRAKINUXIS_Lite - 6S High-Performance FOC BLDC ESC
- moved on the sheet: C1, C12, C13, C14, C15, C26, C27, C28, D1, FB1, J2, LED1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

Commit message: latest files upload
Parts:
- added JP1: BOOT, Jumper:SolderJumper-2_P1.3mm_Open_RoundedPad1.0x1.5mm, symbol Jumper:SolderJumper_2_Open
- C10, C8, C9: value 100nF -> 1uF
Connections:
- net +3V3_SYS: now also JP1.2 (B); no longer C11.2, U6.6 (VDD)
- net BOOT0_GND: now also JP1.1 (A)
- new net: C11.2, U6.6 (VDD)

Commit message: Uploaded all latest files to GitHub
Parts:
- removed R19, R20, R21: 33k, Resistor_SMD:R_0603_1608Metric, symbol Device:R
- added TP1: +3V3_SYS, TestPoint:TestPoint_THTPad_2.0x2.0mm_Drill1.0mm, symbol Connector:TestPoint
- added TP2: SWDIO, TestPoint:TestPoint_THTPad_2.0x2.0mm_Drill1.0mm, symbol Connector:TestPoint
- added TP3: SWCLK, TestPoint:TestPoint_THTPad_2.0x2.0mm_Drill1.0mm, symbol Connector:TestPoint
- added TP4: GND, TestPoint:TestPoint_THTPad_2.0x2.0mm_Drill1.0mm, symbol Connector:TestPoint
- added TP5: NRST, TestPoint:TestPoint_THTPad_2.0x2.0mm_Drill1.0mm, symbol Connector:TestPoint
- C1: value 1000uF -> 1000uF 50V
- C10, C8, C9: value 1uF -> 1uF 50V
- C11, C12, C13, C14, C15, C16, C17, C18: value 100nF -> 100nF 25V
- C19, C2, C20, C21, C22, C3, C4, C5, C6, C7: value 10uF -> 10uF 50V
- C23, C24, C25, C26, C27, C28: value 1uF -> 1uF 16V
- C29, C30, C31, C32, C33, C34: value 1nF -> 1nF 50V
- PAD1, PAD2, PAD3, PAD4, PAD5: footprint Custom_Pads:Pad_10x7mm_WireHole -> TestPoint:TestPoint_THTPad_4.0x4.0mm_Drill2.0mm
- SW1: footprint (none) -> Button_Switch_SMD:SW_SPST_B3S-1000
- U4: value L78L05ABUTR -> DI78M05UAB
- renumbered R12 to R19, R14 to R20, R16 to R21
Connections:
- net +3V3_SYS: now also TP1.1
- net GND: now also TP4.1
- net MCU_RESET: now also TP5.1
- net SWCLK: now also TP3.1
- net SWDIO: now also TP2.1
- net R1_Kelvin (+) renamed SHUNT_U_IN
- net R2_Kelvin (+) renamed SHUNT_V_IN
- net R3_Kelvin (+) renamed SHUNT_W_IN
Other:
- moved on the sheet: C29, C31, LED1, LED2, R27, R28, R29, R30, R31, R32, R37, R38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
