File: hardware/RUDRAKINUXIS_Lite.kicad_pcb (KiCad board)
At the start: 4 copper layers, 65 x 55 mm, 5 parts

Commit message: I uploaded all latest files to GitHub
Parts:
- added C_BULK: 1000uF_50V, Capacitor_THT:CP_Radial_D16.0mm_P7.50mm, F.Cu at (22.0, 20.0)
- BAT+, BAT-, PHASE_U, PHASE_V, PHASE_W: value (none) -> Pad_10x7mm_WireHole
Other:
- net class Default added: clearance 0.15, trace_width 0.20, via_dia 0.60, via_drill 0.30
- net class Power_Heavy added: clearance 0.40, trace_width 2.50, via_dia 0.80, via_drill 0.40

Commit message: Uploading latest files, 50% work done in schematic
Other:
- net class Default removed
- net class Power_Heavy removed
- rule solder_mask_min_width: 0.10 -> 0.1

Commit message: Uploaded all latest files to GitHub
Parts:
- removed BAT+, BAT-, PHASE_U, PHASE_V, PHASE_W: Pad_10x7mm_WireHole, Custom_Pads:Pad_10x7mm_WireHole
- removed C_BULK: 1000uF_50V, Capacitor_THT:CP_Radial_D16.0mm_P7.50mm
- added C1: 1000uF 50V, easyeda2kicad:CAP_16 X 25_PAN, F.Cu at (159.8, 68.4)
- added C10: 1uF 50V, Capacitor_SMD:C_0603_1608Metric, F.Cu at (162.0, 33.0)
- added C11: 100nF 25V, Capacitor_SMD:C_0603_1608Metric, F.Cu at (143.6, 81.5)
- added C12: 100nF 25V, Capacitor_SMD:C_0603_1608Metric, F.Cu at (138.8, 62.0)
- added C13: 100nF 25V, Capacitor_SMD:C_0603_1608Metric, F.Cu at (145.5, 52.5)
- added C14: 100nF 25V, Capacitor_SMD:C_0603_1608Metric, F.Cu at (136.5, 50.0)
- added C15: 100nF 25V, Capacitor_SMD:C_0603_1608Metric, F.Cu at (133.0, 60.0)
- added C16: 100nF 25V, Capacitor_SMD:C_0603_1608Metric, F.Cu at (131.5, 43.5)
- added C17: 100nF 25V, Capacitor_SMD:C_0603_1608Metric, F.Cu at (139.0, 40.0)
- added C18: 100nF 25V, Capacitor_SMD:C_0603_1608Metric, F.Cu at (120.0, 62.5)
- added C19: 10uF 50V, Capacitor_SMD:C_1206_3216Metric, F.Cu at (160.5, 45.2)
- added C2: 10uF 50V, Capacitor_SMD:C_1206_3216Metric, F.Cu at (173.0, 36.6)
- added C20: 10uF 50V, Capacitor_SMD:C_1206_3216Metric, F.Cu at (119.0, 75.0)
- added C21: 10uF 50V, Capacitor_SMD:C_1206_3216Metric, F.Cu at (120.5, 46.5)
- added C22: 10uF 50V, Capacitor_SMD:C_1206_3216Metric, F.Cu at (118.0, 46.5)
- added C23: 1uF 16V, Capacitor_SMD:C_0603_1608Metric, F.Cu at (123.2, 63.0)
- added C24: 1uF 16V, Capacitor_SMD:C_0603_1608Metric, F.Cu at (128.0, 47.5)
- added C25: 1uF 16V, Capacitor_SMD:C_0603_1608Metric, F.Cu at (123.5, 47.5)
- added C26: 1uF 16V, Capacitor_SMD:C_0603_1608Metric, F.Cu at (139.5, 70.0)
- added C27: 1uF 16V, Capacitor_SMD:C_0603_1608Metric, F.Cu at (142.0, 67.0)
- added C28: 1uF 16V, Capacitor_SMD:C_0603_1608Metric, F.Cu at (145.5, 54.2)
- added C29: 1nF 50V, Capacitor_SMD:C_0603_1608Metric, F.Cu at (145.0, 60.2)
- added C3: 10uF 50V, Capacitor_SMD:C_1206_3216Metric, F.Cu at (170.1, 36.7)
- added C30: 1nF 50V, Capacitor_SMD:C_0603_1608Metric, F.Cu at (148.2, 59.5)
- added C31: 1nF 50V, Capacitor_SMD:C_0603_1608Metric, F.Cu at (145.0, 58.4)
- added C32: 1nF 50V, Capacitor_SMD:C_0603_1608Metric, F.Cu at (140.5, 62.8)
- added C33: 1nF 50V, Capacitor_SMD:C_0603_1608Metric, F.Cu at (142.8, 62.5)
- added C34: 1nF 50V, Capacitor_SMD:C_0603_1608Metric, F.Cu at (145.0, 56.5)
- added C4: 10uF 50V, Capacitor_SMD:C_1206_3216Metric, F.Cu at (169.2, 55.9)
- added C5: 10uF 50V, Capacitor_SMD:C_1206_3216Metric, F.Cu at (172.0, 55.9)
- added C6: 10uF 50V, Capacitor_SMD:C_1206_3216Metric, F.Cu at (177.7, 61.6)
- added C7: 10uF 50V, Capacitor_SMD:C_1206_3216Metric, F.Cu at (177.6, 64.3)
- added C8: 1uF 50V, Capacitor_SMD:C_0603_1608Metric, F.Cu at (155.5, 33.0)
- added C9: 1uF 50V, Capacitor_SMD:C_0603_1608Metric, F.Cu at (158.8, 33.0)
- added D1: SMCJ28A, easyeda2kicad:DIODE_DO-214AC, F.Cu at (157.6, 80.4)
- added D2: SS14, Diode_SMD:D_SMA, F.Cu at (136.0, 78.0)
- added D3: SS14, Diode_SMD:D_SMA, F.Cu at (136.5, 69.5)
- added FB1: 600R, Inductor_SMD:L_0603_1608Metric, F.Cu at (144.0, 67.0)
- added J1: USB4105-GF-A, easyeda2kicad:TYPE-C-SMD_SBC-160S1A-20-S412, F.Cu at (128.0, 79.0)
- added J2: SM06B-SRSS-TB, easyeda2kicad:CONN-SMD_SM06B-SRSS-TB-LF-SN, F.Cu at (125.0, 35.0)
- added JP1: BOOT, Jumper:SolderJumper-2_P1.3mm_Open_RoundedPad1.0x1.5mm, F.Cu at (132.4, 63.2)
- added L1: 47uH, easyeda2kicad:IND-SMD_L10.2-W10.0, F.Cu at (123.5, 55.1)
- added LED1: Green, LED_SMD:LED_0603_1608Metric, F.Cu at (147.8, 74.0)
- added LED2: Blue, LED_SMD:LED_0603_1608Metric, F.Cu at (133.0, 67.0)
- added PAD1: BAT+, TestPoint:TestPoint_THTPad_4.0x4.0mm_Drill2.0mm, F.Cu at (176.8, 79.9)
- added PAD2: BAT-, TestPoint:TestPoint_THTPad_4.0x4.0mm_Drill2.0mm, F.Cu at (167.5, 80.2)
- added PAD3: PHASE_U, TestPoint:TestPoint_THTPad_4.0x4.0mm_Drill2.0mm, F.Cu at (191.0, 39.2)
- added PAD4: PHASE_V, TestPoint:TestPoint_THTPad_4.0x4.0mm_Drill2.0mm, F.Cu at (190.7, 55.3)
- added PAD5: PHASE_W, TestPoint:TestPoint_THTPad_4.0x4.0mm_Drill2.0mm, F.Cu at (190.7, 75.5)
- added Q1: NTMFS5H600NLT1G, easyeda2kicad:DFN-5_L5.9-W4.9-P1.27-LS6.2-BL_CASE-488AA, F.Cu at (172.2, 42.8)
- added Q2: NTMFS5H600NLT1G, easyeda2kicad:DFN-5_L5.9-W4.9-P1.27-LS6.2-BL_CASE-488AA, F.Cu at (183.0, 35.3)
- added Q3: NTMFS5H600NLT1G, easyeda2kicad:DFN-5_L5.9-W4.9-P1.27-LS6.2-BL_CASE-488AA, F.Cu at (170.0, 49.9)
- added Q4: NTMFS5H600NLT1G, easyeda2kicad:DFN-5_L5.9-W4.9-P1.27-LS6.2-BL_CASE-488AA, F.Cu at (183.2, 47.6)
- added Q5: NTMFS5H600NLT1G, easyeda2kicad:DFN-5_L5.9-W4.9-P1.27-LS6.2-BL_CASE-488AA, F.Cu at (179.7, 56.6)
- added Q6: NTMFS5H600NLT1G, easyeda2kicad:DFN-5_L5.9-W4.9-P1.27-LS6.2-BL_CASE-488AA, F.Cu at (185.2, 65.1)
- added R1: 0.5m, Resistor_SMD:R_2512_6332Metric, F.Cu at (190.1, 47.4)
- added R10: 10k, Resistor_SMD:R_0603_1608Metric, F.Cu at (167.4, 41.5)
- added R11: 10k, Resistor_SMD:R_0603_1608Metric, F.Cu at (178.0, 33.5)
- added R12: 10k, Resistor_SMD:R_0603_1608Metric, F.Cu at (174.5, 50.4)
- added R13: 10k, Resistor_SMD:R_0603_1608Metric, F.Cu at (179.3, 48.9)
- added R14: 10k, Resistor_SMD:R_0603_1608Metric, F.Cu at (183.5, 55.1)
- added R15: 10k, Resistor_SMD:R_0603_1608Metric, F.Cu at (184.3, 61.2)
- added R16: 10k, Resistor_SMD:R_0603_1608Metric, F.Cu at (133.5, 52.2)
- added R17: 10k, Resistor_SMD:R_0603_1608Metric, F.Cu at (133.2, 57.5)
- added R18: 10k, Resistor_SMD:R_0603_1608Metric, F.Cu at (141.2, 50.2)
- added R19: 33k, Resistor_SMD:R_0603_1608Metric, F.Cu at (148.2, 64.8)
- added R2: 0.5m, Resistor_SMD:R_2512_6332Metric, F.Cu at (179.1, 42.5)
- added R20: 33k, Resistor_SMD:R_0603_1608Metric, F.Cu at (154.3, 61.5)
- added R21: 33k, Resistor_SMD:R_0603_1608Metric, F.Cu at (152.6, 55.0)
- added R22: 33k, Resistor_SMD:R_0603_1608Metric, F.Cu at (172.3, 79.2)
- added R23: 3.3k, Resistor_SMD:R_0603_1608Metric, F.Cu at (148.2, 63.0)
- added R24: 3.3k, Resistor_SMD:R_0603_1608Metric, F.Cu at (148.2, 61.2)
- added R25: 3.3k, Resistor_SMD:R_0603_1608Metric, F.Cu at (149.2, 57.5)
- added R26: 3.3k, Resistor_SMD:R_0603_1608Metric, F.Cu at (139.7, 50.2)
- added R27: 100R, Resistor_SMD:R_0603_1608Metric, F.Cu at (193.0, 46.5)
- added R28: 100R, Resistor_SMD:R_0603_1608Metric, F.Cu at (182.0, 82.2)
- added R29: 100R, Resistor_SMD:R_0603_1608Metric, F.Cu at (177.7, 48.6)
- added R3: 0.5m, Resistor_SMD:R_2512_6332Metric, F.Cu at (190.7, 67.6)
- added R30: 100R, Resistor_SMD:R_0603_1608Metric, F.Cu at (185.3, 82.2)
- added R31: 100R, Resistor_SMD:R_0603_1608Metric, F.Cu at (192.9, 61.3)
- added R32: 100R, Resistor_SMD:R_0603_1608Metric, F.Cu at (188.6, 82.2)
- added R33: 5.1k, Resistor_SMD:R_0603_1608Metric, F.Cu at (125.0, 73.0)
- added R34: 5.1k, Resistor_SMD:R_0603_1608Metric, F.Cu at (131.0, 73.0)
- added R35: 100k, Resistor_SMD:R_0603_1608Metric, F.Cu at (127.0, 64.0)
- added R36: 11k, Resistor_SMD:R_0603_1608Metric, F.Cu at (125.0, 66.0)
- added R37: 1k, Resistor_SMD:R_0603_1608Metric, F.Cu at (144.5, 74.5)
- added R38: 1k, Resistor_SMD:R_0603_1608Metric, F.Cu at (137.0, 62.0)
- added R39: 120R, Resistor_SMD:R_0805_2012Metric, F.Cu at (135.2, 38.2)
- added R4: 10, Resistor_SMD:R_0603_1608Metric, F.Cu at (167.4, 44.8)
- added R40: 33k, Resistor_SMD:R_1206_3216Metric, F.Cu at (162.3, 79.9)
- added R5: 10, Resistor_SMD:R_0603_1608Metric, F.Cu at (177.8, 37.2)
- added R6: 10, Resistor_SMD:R_0603_1608Metric, F.Cu at (174.3, 47.9)
- added R7: 10, Resistor_SMD:R_0603_1608Metric, F.Cu at (182.0, 42.1)
- added R8: 10, Resistor_SMD:R_0603_1608Metric, F.Cu at (185.5, 55.2)
- added R9: 10, Resistor_SMD:R_0603_1608Metric, F.Cu at (186.9, 60.4)
- added SW1: B3S-1000P, Button_Switch_SMD:SW_SPST_B3S-1000, F.Cu at (147.8, 40.5)
- added TH1: 10k NTC, Resistor_SMD:R_0603_1608Metric, F.Cu at (143.0, 50.5)
- added TP1: +3V3_SYS, TestPoint:TestPoint_THTPad_2.0x2.0mm_Drill1.0mm, F.Cu at (135.0, 33.0)
- added TP2: SWDIO, TestPoint:TestPoint_THTPad_2.0x2.0mm_Drill1.0mm, F.Cu at (138.2, 33.0)
- added TP3: SWCLK, TestPoint:TestPoint_THTPad_2.0x2.0mm_Drill1.0mm, F.Cu at (141.5, 33.0)
- added TP4: GND, TestPoint:TestPoint_THTPad_2.0x2.0mm_Drill1.0mm, F.Cu at (144.8, 33.0)
- added TP5: NRST, TestPoint:TestPoint_THTPad_2.0x2.0mm_Drill1.0mm, F.Cu at (148.0, 33.0)
- added U1: STM32G431CBU6, easyeda2kicad:VQFN-48_L7.0-W7.0-P0.50-BL-EP5.5, F.Cu at (139.0, 56.0)
- added U2: DRV8300DPWR, easyeda2kicad:TSSOP-20_L6.5-W4.4-P0.65-LS6.4-BL, F.Cu at (159.0, 38.8)
- added U3: LMR36510ADDAR, easyeda2kicad:SOP-8_L5.0-W4.0-P1.27-LS6.2-BL-EP, F.Cu at (121.0, 68.0)
- added U4: DI78M05UAB, easyeda2kicad:SOT-89-3_L4.5-W2.5-P1.50-LS4.2-TL, F.Cu at (126.5, 44.1)
- added U5: AP2112K-3.3, easyeda2kicad:SOT-25-5_L2.9-W1.6-P0.95-LS2.8-BL, F.Cu at (142.0, 70.5)
- added U6: CP2102N, easyeda2kicad:QFN-24_L4.0-W4.0-P0.50-TL-EP2.6, F.Cu at (148.0, 78.0)
- added U7: TJA1051T/3,118, easyeda2kicad:SOIC-8_L4.9-W3.9-P1.27-LS6.0-BL, F.Cu at (135.0, 43.8)
- added U8: USBLC6-2SC6, easyeda2kicad:SOT-23-6_L2.9-W1.6-P0.95-LS2.8-BL, F.Cu at (141.0, 78.0)
- added U9: ESDCAN24-2BLY, easyeda2kicad:SOT_24-2BLY_STM, F.Cu at (119.5, 41.8)
Routing:
- net /V_BAT: track 0.00 -> 221.1 mm, vias 0 -> 16
- net GND: track 0.00 -> 131.7 mm, vias 0 -> 99
- net /+3V3_SYS: track 0.00 -> 120.3 mm, vias 0 -> 11
- net /ISENSE_U: track 0.00 -> 112.8 mm, vias 0 -> 4
- net /+10V_GATE: track 0.00 -> 101.1 mm, vias 0 -> 4
- net /ISENSE_W: track 0.00 -> 100.3 mm, vias 0 -> 4
- net /VBAT_SENSE: track 0.00 -> 74.9 mm, vias 0 -> 6
- net /SW1_TEST: track 0.00 -> 74.9 mm, vias 0 -> 2
- net /MCU_UART_TX: track 0.00 -> 72.0 mm, vias 0 -> 3
- net /MOTOR_U: track 0.00 -> 70.2 mm, vias 0 -> 5
- net /ISENSE_V: track 0.00 -> 60.9 mm, vias 0 -> 4
- net /GATE_HW_DRV: track 0.00 -> 58.6 mm, vias 0 -> 4
- net /GATE_HV_DRV: track 0.00 -> 57.7 mm, vias 0 -> 4
- net /+5V_AUX: track 0.00 -> 56.1 mm
- net /MOTOR_V: track 0.00 -> 53.7 mm, vias 0 -> 2
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Other:
- board size 65 x 55 mm -> 78.5 x 55 mm
- rule solder_mask_min_width: 0.1 -> 0.5

Commit message: uploaded all latest files.
Parts:
- moved PAD3 0.60 mm to (190.4, 39.2)
- moved Q2 0.19 mm to (182.8, 35.3)
- moved C27 0.10 mm to (142.0, 66.9)
- moved FB1 0.10 mm to (144.0, 66.9)
Connections:
- J1 pad : (no net) -> GND
Routing:
- net /V_BAT: track 221.1 -> 226.0 mm
- net /MOTOR_V: track 53.7 -> 56.3 mm
- net /MOTOR_U: track 70.2 -> 72.7 mm, vias 5 -> 6
- net /+3V3_SYS: track 120.3 -> 122.6 mm
- net GND: track 131.7 -> 129.5 mm, vias 99 -> 95
- net Net-(Q2-G): track 6.33 -> 7.44 mm
- net /IN_HW: track 25.8 -> 26.6 mm
- net /SWCLK: track 31.7 -> 32.2 mm
- net /IN_LV: track 33.0 -> 33.5 mm
- net /ISENSE_W: track 100.3 -> 100.7 mm, vias 4 -> 3
- net /IN_LW: track 34.5 -> 34.6 mm, vias 5 -> 4
- added copper zone on B.Cu, net GND
- added copper zone on In1.Cu, net GND
- added copper zone on In2.Cu, net GND
Other:
- outline, holes or cut-outs redrawn
